File: Electronique/boardDesign/IHM2/IHM2.kicad_sch (KiCad schematic)
At the start: 0 parts

Commit message: doc : remade graphs for PID in file to show that Td = 1000 in the related simulations feat : footprints and schematic for HMI done
Parts:
- added D1, D2, D3, D4: LED, LED_SMD:LED_1206_3216Metric, symbol Device:LED
- added J1: Conn_01x14, rotaryEncoder:1x14 THT input, symbol Connector_Generic:Conn_01x14
- added R1, R2, R3, R4: 220, PCM_4ms_Resistor:R_0805_2012Metric, symbol Device:R
- added SW1: SW_Push_Dual_INIT, rotaryEncoder:SW_Push_Dual_13mm, symbol Switch:SW_Push_Dual
- added SW2: SW_Push_Dual_START, rotaryEncoder:SW_Push_Dual_13mm, symbol Switch:SW_Push_Dual
- added SW3: SW_Push_Dual_PAUSE, rotaryEncoder:SW_Push_Dual_13mm, symbol Switch:SW_Push_Dual
- added SW4: RotaryEncoder_Switch, rotaryEncoder:RotaryEncoder_SW, symbol rotaryEncoder:RotaryEncoder_Switch
- added U1: ER_OLEDM0.91_1x-I2C, rotaryEncoder:oledDisplay1Inch, symbol Display_Graphic:ER_OLEDM0.91_1x-I2C
Connections:
- new net: D4.2 (A), R4.2
- new net: D3.2 (A), R3.2
- new net: D1.2 (A), R1.2
- new net: D2.2 (A), R2.2
- new net +5V: J1.1 (Pin_1), SW4.4 (S1), U1.2 (VCC)
- new net CLK_ROT: J1.3 (Pin_3), SW4.1 (CLK)
- new net DT_ROT: J1.4 (Pin_4), SW4.2 (DT)
- new net GND: D1.1 (K), D2.1 (K), D3.1 (K), D4.1 (K), J1.2 (Pin_2), SW1.2, SW2.2, SW3.2, SW4.5 (S2), U1.1 (GND)
- new net LED_INIT: J1.9 (Pin_9), R2.1
- new net LED_PAUSE: J1.11 (Pin_11), R4.1
- new net LED_POW: J1.8 (Pin_8), R1.1
- new net LED_START: J1.10 (Pin_10), R3.1
- new net SCL_SCREEN: J1.6 (Pin_6), U1.3 (SCL)
- new net SDA_SCREEN: J1.7 (Pin_7), U1.4 (SDA)
- new net SW_INIT_OUT: J1.12 (Pin_12), SW1.1
- new net SW_PAUSE_OUT: J1.14 (Pin_14), SW3.1
- new net SW_ROT: J1.5 (Pin_5), SW4.3 (SW)
- new net SW_START_OUT: J1.13 (Pin_13), SW2.1
- no-connect marks 0 -> 6
Other:
- company: (none) -> MECA22-3
- title: (none) -> CobotBoy_IHM
